File: PCB/Quantum-MINI.kicad_pcb (KiCad board)
At the start: 2 copper layers, 250.6 x 162.2 mm, 80 parts, among them J1 USB C Connector, J2 JTAG_TC2030, SW1 Boot, SW10 MX_SW_HS, SW11 MX_SW_solder, SW12 MX_SW_solder, SW13 MX_SW_HS, SW14 MX_SW_solder, SW15 MX_SW_HS, SW16 MX_SW_solder, SW17 MX_SW_HS, SW18 MX_SW_HS, SW19 MX_SW_solder, SW2 MX_SW_HS, SW20 MX_SW_HS, SW21 MX_SW_solder, SW22 MX_SW_solder, SW23 MX_SW_HS, SW24 MX_SW_HS, SW25 MX_SW_solder, SW26 MX_SW_HS, SW27 MX_SW_solder, SW28 MX_SW_HS, SW29 MX_SW_solder, SW3 MX_SW_solder, SW30 MX_SW_solder, SW31 MX_SW_HS, SW32 MX_SW_HS, SW33 MX_SW_solder, SW34 MX_SW_solder, SW35 MX_SW_HS, SW36 MX_SW_HS, SW37 MX_SW_solder, SW38 MX_SW_solder, SW39 MX_SW_HS, SW4 MX_SW_HS, SW40 MX_SW_HS, SW41 MX_SW_solder, SW5 MX_SW_solder, SW6 MX_SW_solder, SW7 MX_SW_HS, SW8 MX_SW_solder, SW9 MX_SW_HS, U1 XC6206, U2 USBLC6-2SC6, U3 RP2040, U4 W25Q128JVS, Y1 12MHz

Commit message: Decided to use a daughterboard
- Removed USB port
- Re-arranged rp2040 circuit
- Added USB passthrough
- Adjusted board outline
Parts:
- removed D2: Schottky Diode, Diode_SMD:D_SOD-123
- removed F1: 500 mA, Fuse:Fuse_1206_3216Metric
- removed J1: USB C Connector, footprints:TYPE-C_24P_QCHT
- removed R1: 1M, Resistor_SMD:R_0603_1608Metric
- removed R2, R3: 5.1k, Resistor_SMD:R_0402_1005Metric
- removed U2: USBLC6-2SC6, Package_TO_SOT_SMD:SOT-23-6
- added C18: 4.7uf, Capacitor_SMD:C_0603_1608Metric, F.Cu at (26.7, 28.7)
- added C19: 100nF, Capacitor_SMD:C_0402_1005Metric, F.Cu at (-20.1, 37.1)
- added F2: 500 mA, Fuse:Fuse_1206_3216Metric, F.Cu at (49.1, 30.6)
- added J3: USB_A, USB1130-15-A:GCT_USB1130-15-A_REVA, F.Cu at (37.1, 27.9)
- added J4: Conn_01x06, Connector_PinSocket_2.54mm:PinSocket_1x06_P2.54mm_Horizontal, F.Cu at (154.8, 55.0)
- added R12: 1M, Resistor_SMD:R_0603_1608Metric, F.Cu at (26.7, 27.2)
- added R13: 10k, Resistor_SMD:R_0402_1005Metric, F.Cu at (-30.5, 37.1)
- added R14: 22, Resistor_SMD:R_0603_1608Metric, F.Cu at (53.6, 23.0)
- added R15: 22, Resistor_SMD:R_0603_1608Metric, F.Cu at (53.6, 24.5)
- added SW42: SW_SPDT, Button_Switch_SMD:SW_SPDT_PCM12, F.Cu at (99.8, 5.67)
- added U5: USBLC6-2SC6, Package_TO_SOT_SMD:SOT-23-6, F.Cu at (47.7, 23.7)
- added U6: W25Q128JVS, Package_SO:SOIC-8_5.23x5.23mm_P1.27mm, F.Cu at (-25.3, 39.5)
- R10: value 1k -> 10k
- moved U4 167.0 mm to (-26.2, 51.1), turned to -90 degrees
- moved R10 159.6 mm to (-22.4, 47.5), turned to 180 degrees
- moved SW1 157.2 mm to (-17.1, 49.3), turned to 180 degrees
- moved J2 79.1 mm to (78.6, 39.2), turned to 180 degrees
- moved C8 74.5 mm to (78.7, 33.0), turned to 0 degrees
- moved R7 73.1 mm to (82.8, 37.9), turned to 90 degrees
- moved Y1 72.4 mm to (78.7, 29.7), turned to 90 degrees
- moved C6 71.1 mm to (82.2, 34.4), turned to 180 degrees
- moved C7 70.9 mm to (78.4, 26.2), turned to 180 degrees
- moved D3 70.5 mm to (90.7, 42.8), turned to 90 degrees
- moved C14 70.0 mm to (82.2, 32.9), turned to 180 degrees
- moved C11 69.7 mm to (86.9, 39.3), turned to -135 degrees
- moved R11 68.6 mm to (82.2, 30.8), turned to 0 degrees
- moved R4 67.9 mm to (90.7, 40.2), turned to -90 degrees
- moved R6 66.0 mm to (95.1, 44.0), turned to 0 degrees
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Connections:
- R10 pad 1: /~{USB_BOOT} -> MB1
- R10 pad 2: CS -> +3V3
- SW1 pad 2: /~{USB_BOOT} -> CS
- U3 pad 13: unconnected-(U3-GPIO10-Pad13) -> USBD+
- U3 pad 14: unconnected-(U3-GPIO11-Pad14) -> USBD-
- U4 pad 1: CS -> MB1
Routing:
- net D+: track 7.30 -> 65.3 mm
- net D-: track 7.38 -> 63.3 mm
- net USBD+: track 0.00 -> 38.8 mm
- net USBD-: track 0.00 -> 38.1 mm
- net 3vCable: track 34.8 -> 0.00 mm, vias 2 -> 0
- net DATA: track 53.6 -> 26.0 mm, vias 2 -> 1
- net Net-(J1-SHIELD): track 23.5 -> 0.00 mm
- net Net-(J3-Shield): track 0.00 -> 18.2 mm
- net USBDBUS+: track 0.00 -> 17.0 mm
- net USBDBUS-: track 0.00 -> 16.3 mm
- net Net-(J1-CC2): track 15.6 -> 0.00 mm
- net USBVBUS: track 0.00 -> 14.9 mm
- net A: track 16.0 -> 30.4 mm
- net C_DN: track 15.1 -> 29.5 mm
- net CS: track 20.7 -> 6.52 mm
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Other:
- board size 250.6 x 162.2 mm -> 250.6 x 155.2 mm
